File: AN108 Bridge/an108_bridge.kicad_pcb (KiCad board)
At the start: 2 copper layers, 31 x 47.8 mm, 5 parts, among them J1 AN108 Header, J2 AD PMOD, J3 DA_PMOD, J4 Conn_01x02, J5 Conn_01x02

Commit message: Swapped +5v and GND on AN108 header
Connections:
- J1 pad 1: +5V -> GND
- J1 pad 2: GND -> +5V
Routing:
- net +5V: track 20.8 -> 19.4 mm
Other:
- board text added: "+5"
- board text added: "GND"
Changed lines of the file:
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@@
 			)
 		)
+		(property ki_fp_filters "Connector*:*_2x??_*")
+		(sheetname "Root")
+		(sheetfile "an108_bridge.kicad_sch")
 		(attr through_hole)
 		(fp_line
@@
 			)
 		)
+		(property ki_fp_filters "Connector*:*_2x??_*")
+		(sheetname "Root")
+		(sheetfile "an108_bridge.kicad_sch")
 		(attr through_hole)
 		(fp_line
@@
 			(layers "*.Cu" "*.Mask")
 			(remove_unused_layers no)
-			(net 6 "+5V")
+			(net 4 "GND")
 			(pinfunction "Pin_1")
 			(pintype "passive")
@@
 			(layers "*.Cu" "*.Mask")
 			(remove_unused_layers no)
-			(net 4 "GND")
+			(net 6 "+5V")
 			(pinfunction "Pin_2")
 			(pintype "passive")
@@
 			)
 		)
+		(property ki_fp_filters "Connector*:*_1x??_*")
+		(sheetname "Root")
+		(sheetfile "an108_bridge.kicad_sch")
 		(attr through_hole)
 		(fp_line
@@
 			)
 		)
+		(property ki_fp_filters "Connector*:*_1x??_*")
+		(sheetname "Root")
+		(sheetfile "an108_bridge.kicad_sch")
 		(attr through_hole)
 		(fp_line
@@
 			)
 		)
+		(property ki_fp_filters "Connector*:*_2x??_*")
+		(sheetname "Root")
+		(sheetfile "an108_bridge.kicad_sch")
 		(attr through_hole)
 		(fp_line
@@
 			)
 		)
+	)
+	(gr_rect
+		(start 147.25 98)
+		(end 153.75 110.5)
+		(stroke
+			(width 0.1)
+			(type default)
+		)
+		(fill none)
+		(layer "F.SilkS")
+	)
+	(gr_rect
+		(start 147.25 77.5)
+		(end 153.5 90.25)
+		(stroke
+			(width 0.1)
+			(type default)
+		)
+		(fill none)
+		(layer "F.SilkS")
 	)
 	(gr_rect
@@
 		)
 	)
+	(gr_text "+5"
+		(at 130.575 112.745 0)
+		(layer "F.SilkS")
+		(effects
+			(font
+				(size 1 1)
+				(thickness 0.2)
+				(bold yes)
+			)
+			(justify left bottom)
+		)
+	)
 	(gr_text "AN108 Header"
 		(at 156.5 114 90)
@@
 		)
 	)
+	(gr_text "GND"
+		(at 127.5 112.745 0)
+		(layer "F.SilkS")
+		(effects
+			(font
+				(size 1 1)
+				(thickness 0.2)
+				(bold yes)
+			)
+			(justify left bottom)
+		)
+	)
 	(gr_text "1"
 		(at 153.565 115.045 0)
@@
 	)
 	(segment
-		(start 150.365 115.67)
-		(end 151.665 114.37)
+		(start 149 116)
+		(end 149 114.495)
 		(width 0.5)
 		(layer "F.Cu")
@@
 	)
 	(segment
-		(start 132.975 115.67)
-		(end 150.365 115.67)
+		(start 149 114.495)
+		(end 149.125 114.37)
 		(width 0.5)
 		(layer "F.Cu")
@@
 	(segment
 		(start 131.85 114.545)
-		(end 132.975 115.67)
+		(end 133.305 116)
 		(width 0.5)
 		(layer "F.Cu")
+		(net 6)
+	)
+	(segment
+		(start 133.305 116)
+		(end 149 116)
+		(width 0.5)
+		(layer "F.Cu")
